Commit message: [ARM-44] Correction des frames TF

File: Dev_code_version_SITL/ros_catkin_ws/src/ardupilot_sitl_gazebo_plugin/ardupilot_sitl_gazebo_plugin/urdf/armada.xacro (robot description, xacro)
@@ -2,5 +2,5 @@
 <robot name="armada" xmlns:xacro="http://ros.org/wiki/xacro">
   <!-- Properties -->
-  <xacro:property name="namespace" value="erlecopter" />
+  <xacro:property name="namespace" value="" />
   <xacro:property name="rotor_velocity_slowdown_sim" value="10" />
   <xacro:property name="mesh_file" value="erlecopter.dae" />
@@ -58,96 +58,4 @@
   </xacro:multirotor_base_macro>
   <xacro:property name="M_PI" value="3.1415926535897931" />
-  <!-- Sonar sensor
- <xacro:include filename="$(find ardupilot_sitl_gazebo_plugin)/urdf/sensors/real_sonar_sensor.urdf.xacro" />-->
-  <!-- Configuration SIDE
-  <xacro:real_sonar_sensor
-    name="real_sonar_front"
-    parent="base_link"
-    ros_topic="sonar_front"
-    update_rate="10"
-    min_range="0.02"
-    max_range="7.65"
-    radius="2.3"
-    sensor_mesh="max_sonar_ez4/meshes/max_sonar_ez4.dae">
-    <origin xyz="0.1 0 0" rpy="0 ${270*M_PI/180} 0"/>
-  </xacro:real_sonar_sensor>
-  <xacro:real_sonar_sensor
-    name="real_sonar_down"
-    parent="base_link"
-    ros_topic="sonar_down"
-    update_rate="10"
-    min_range="0.02"
-    max_range="7.65"
-    radius="2.3"
-    sensor_mesh="max_sonar_ez4/meshes/max_sonar_ez4.dae">
-    <origin xyz="-0.1 0 0" rpy="0 ${90*M_PI/180} 0"/>
-  </xacro:real_sonar_sensor>
-  <xacro:real_sonar_sensor
-    name="real_sonar_right"
-    parent="base_link"
-    ros_topic="sonar_right"
-    update_rate="10"
-    min_range="0.02"
-    max_range="7.65"
-    radius="2.3"
-    sensor_mesh="max_sonar_ez4/meshes/max_sonar_ez4.dae">
-    <origin xyz="0 -0.1 0" rpy="${270*M_PI/180} 0 0 "/>
-  </xacro:real_sonar_sensor>
-  <xacro:real_sonar_sensor
-    name="real_sonar_left"
-    parent="base_link"
-    ros_topic="sonar_left"
-    update_rate="10"
-    min_range="0.02"
-    max_range="7.65"
-    radius="2.3"
-    sensor_mesh="max_sonar_ez4/meshes/max_sonar_ez4.dae">
-    <origin xyz="0 0.1 0" rpy="${90*M_PI/180} 0 0"/>
-  </xacro:real_sonar_sensor> -->
-  <!-- Configuration FEET
-  <xacro:real_sonar_sensor
-    name="real_sonar_front_left"
-    parent="base_link"
-    ros_topic="sonar_front_left"
-    update_rate="10"
-    min_range="0.02"
-    max_range="7.65"
-    radius="2.3"
-    sensor_mesh="max_sonar_ez4/meshes/max_sonar_ez4.dae">
-    <origin xyz="0.15 0.15 -0.03" rpy="0 ${270*M_PI/180} ${45*M_PI/180}"/>
-  </xacro:real_sonar_sensor>
-  <xacro:real_sonar_sensor
-    name="real_sonar_back_right"
-    parent="base_link"
-    ros_topic="sonar_back_right"
-    update_rate="10"
-    min_range="0.02"
-    max_range="7.65"
-    radius="2.3"
-    sensor_mesh="max_sonar_ez4/meshes/max_sonar_ez4.dae">
-    <origin xyz="-0.15 -0.15 -0.03" rpy="0 ${90*M_PI/180} ${45*M_PI/180}"/>
-  </xacro:real_sonar_sensor>
-  <xacro:real_sonar_sensor
-    name="real_sonar_front_right"
-    parent="base_link"
-    ros_topic="sonar_front_right"
-    update_rate="10"
-    min_range="0.02"
-    max_range="7.65"
-    radius="2.3"
-    sensor_mesh="max_sonar_ez4/meshes/max_sonar_ez4.dae">
-    <origin xyz="0.15 -0.15 -0.03" rpy="${270*M_PI/180} 0 ${45*M_PI/180} "/>
-  </xacro:real_sonar_sensor>
-  <xacro:real_sonar_sensor
-    name="real_sonar_back_left"
-    parent="base_link"
-    ros_topic="sonar_back_left"
-    update_rate="10"
-    min_range="0.02"
-    max_range="7.65"
-    radius="2.3"
-    sensor_mesh="max_sonar_ez4/meshes/max_sonar_ez4.dae">
-    <origin xyz="-0.15 0.15 -0.03" rpy="${90*M_PI/180} 0 ${45*M_PI/180}"/>
-  </xacro:real_sonar_sensor> -->
   <!-- Lidar sensor -->
   <xacro:include filename="$(find ardupilot_sitl_gazebo_plugin)/urdf/sensors/lidar_sensor.urdf.xacro" />
@@ -155,19 +63,18 @@
     name="lidar"
     parent="base_link"
-    ros_topic="lidar"
     update_rate="10"
-    min_range="0.01"
-    max_range="10.0"
+    min_range="0.06"
+    max_range="20.0"
     field_of_view_horizontal="${2*M_PI}"
     field_of_view_vertical="${1*M_PI/180}"
-    ray_count_horizontal="360"
-    ray_count_vertical="1"
-    sensor_mesh_base_1="velodyne_VLP16/meshes/VLP16_base_1.dae"
-    sensor_mesh_base_2="velodyne_VLP16/meshes/VLP16_base_2.dae"
-    sensor_mesh_scan="velodyne_VLP16/meshes/VLP16_scan.dae">
+    ray_count_horizontal="768"
+    ray_count_vertical="2"
+    sensor_mesh_base_1="$(find ardupilot_sitl_gazebo_plugin)/meshes/meshes_sensors/velodyne_VLP16/meshes/VLP16_base_1.dae"
+    sensor_mesh_base_2="$(find ardupilot_sitl_gazebo_plugin)/meshes/meshes_sensors/velodyne_VLP16/meshes/VLP16_base_2.dae"
+    sensor_mesh_scan="$(find ardupilot_sitl_gazebo_plugin)/meshes/meshes_sensors/velodyne_VLP16/meshes/VLP16_scan.dae">
     <origin xyz="0.0 0.0 0.06" rpy="0 0 0"/>
   </xacro:lidar_sensor>
   <!-- Front facing camera -->
-<xacro:include filename="$(find ardupilot_sitl_gazebo_plugin)/urdf/sensors/generic_camera.urdf.xacro" />
+<!-- <xacro:include filename="$(find ardupilot_sitl_gazebo_plugin)/urdf/sensors/generic_camera.urdf.xacro" />
   <xacro:generic_camera
     name="erlecopter/front"
@@ -182,5 +89,5 @@
     framename="erlecopter_frontcam">
     <origin xyz="0.1 0.0 0.05" rpy="0 0 0"/>
-</xacro:generic_camera>
+</xacro:generic_camera>  -->
   <!-- Instantiate rotors -->
   <xacro:vertical_rotor
@@ -246,5 +153,6 @@
     <xacro:insert_block name="rotor_inertia" />
   </xacro:vertical_rotor>
-  <xacro:vertical_rotor robot_namespace="${namespace}"
+  <xacro:vertical_rotor
+    robot_namespace="${namespace}"
     suffix="back_right"
     direction="cw"

File: Dev_code_version_SITL/ros_catkin_ws/src/ardupilot_sitl_gazebo_plugin/ardupilot_sitl_gazebo_plugin/urdf/armada_base.xacro (robot description, xacro)
@@ -1,4 +1,5 @@
 <?xml version="1.0"?>
 <robot name="armada" xmlns:xacro="http://ros.org/wiki/xacro">
+  <xacro:property name="namespace" value="" />
   <xacro:include filename="$(find rotors_description)/urdf/component_snippets.xacro" />
   <!-- Instantiate armada "mechanics" -->
@@ -9,12 +10,12 @@
        We do not use it for we would loose the match X=North, Y=West -->
   <!-- in degrees, 0 so North is towards positive X values, and East is towards negative Y values -->
-  <xacro:property name="referenceHeading" value="0" />
+    <xacro:property name="referenceHeading" value="0" />
   <!-- Instantiate a controller. -->
-  <xacro:controller_plugin_macro
+ <xacro:controller_plugin_macro
     namespace="${namespace}"
     imu_sub_topic="imu"
     >
   </xacro:controller_plugin_macro>
-  <!-- Mount an ADIS16448 IMU. -->
+  <!-- Mount an ADIS16448 IMU.  -->
   <xacro:imu_plugin_macro
     namespace="${namespace}"
@@ -77,5 +78,5 @@
     </plugin>
   </gazebo>
-  <xacro:if value="$(arg enable_ground_truth)">
+   <xacro:if value="$(arg enable_ground_truth)">
     <!-- Mount an IMU providing ground truth. -->
     <xacro:imu_plugin_macro
@@ -97,8 +98,8 @@
       <origin xyz="0 0 0" rpy="0 0 0" />
     </xacro:imu_plugin_macro>
-    <!-- Mount a generic odometry sensor providing ground truth. -->s
+    <!-- Mount a generic odometry sensor providing ground truth. -->
     <xacro:odometry_plugin_macro
-      namespace="${namespace}/ground_truth"
-      odometry_sensor_suffix="gt"
+      namespace="${namespace}"
+      odometry_sensor_suffix=""
       parent_link="base_link"
       pose_topic="pose"
@@ -107,5 +108,5 @@
       transform_topic="transform"
       odometry_topic="odometry"
-      parent_frame_id="odom"
+      parent_frame_id="world"
       mass_odometry_sensor="0.00001"
       measurement_divisor="1"
@@ -124,5 +125,5 @@
       image_scale=""
     >
-      <inertia ixx="0.00001" ixy="0.0" ixz="0.0" iyy="0.00001" iyz="0.0" izz="0.00001" /> <!-- [kg.m^2] [kg.m^2] [kg.m^2] [kg.m^2] [kg.m^2] [kg.m^2] -->
+      <inertia ixx="0.00001" ixy="0.0" ixz="0.0" iyy="0.00001" iyz="0.0" izz="0.00001" /> --> <!-- [kg.m^2] [kg.m^2] [kg.m^2] [kg.m^2] [kg.m^2] [kg.m^2] -->
       <origin xyz="0.0 0.0 0.0" rpy="0.0 0.0 0.0" />
     </xacro:odometry_plugin_macro>

File: Dev_code_version_SITL/ros_catkin_ws/src/ardupilot_sitl_gazebo_plugin/ardupilot_sitl_gazebo_plugin/urdf/sensors/kinect.urdf.xacro (robot description, xacro)
@@ -31,5 +31,5 @@
        <origin xyz="0 0 0" rpy="0 0 ${M_PI/2}"/>
         <geometry>
-         <mesh filename="package://ardupilot_sitl_gazebo_plugin/meshes/meshes_sensors/kinect/kinect.dae"/>
+         <mesh filename="file://ardupilot_sitl_gazebo_plugin/meshes/meshes_sensors/kinect/kinect.dae"/>
         </geometry>
       </visual>

File: Dev_code_version_SITL/ros_catkin_ws/src/ardupilot_sitl_gazebo_plugin/ardupilot_sitl_gazebo_plugin/urdf/sensors/lidar_sensor.urdf.xacro (robot description, xacro)
@@ -1,5 +1,5 @@
 <?xml version="1.0"?>
 <robot xmlns:xacro="http://ros.org/wiki/xacro">
-  <xacro:macro name="lidar_sensor" params="name parent *origin ros_topic update_rate min_range max_range field_of_view_horizontal field_of_view_vertical ray_count_horizontal ray_count_vertical sensor_mesh_base_1 sensor_mesh_base_2 sensor_mesh_scan">
+  <xacro:macro name="lidar_sensor" params="name parent *origin update_rate min_range max_range field_of_view_horizontal field_of_view_vertical ray_count_horizontal ray_count_vertical sensor_mesh_base_1 sensor_mesh_base_2 sensor_mesh_scan">
     <joint name="${name}_joint" type="fixed">
       <xacro:insert_block name="origin" />
@@ -19,5 +19,5 @@
           <!-- <mesh filename="package://rotors_description/meshes/sonar_sensor/max_sonar_ez4.dae"/> -->
           <!--<mesh filename="package://ardupilot_sitl_gazebo_plugin/meshes/${sensor_mesh}"/>-->
-           <mesh filename="model://${sensor_mesh_base_1}"/>
+           <mesh filename="file://${sensor_mesh_base_1}"/>
          <!-- <mesh filename="package://ardupilot_sitl_gazebo_plugin/meshes/meshes_sensor/lidar_lite_v2/meshes/lidar_lite_v2.dae"/> -->
         </geometry>
@@ -29,5 +29,5 @@
           <!-- <mesh filename="package://rotors_description/meshes/sonar_sensor/max_sonar_ez4.dae"/> -->
           <!--<mesh filename="package://ardupilot_sitl_gazebo_plugin/meshes/${sensor_mesh}"/>-->
-           <mesh filename="model://${sensor_mesh_base_2}"/>
+           <mesh filename="file://${sensor_mesh_base_2}"/>
          <!-- <mesh filename="package://ardupilot_sitl_gazebo_plugin/meshes/meshes_sensor/lidar_lite_v2/meshes/lidar_lite_v2.dae"/> -->
         </geometry>
@@ -39,5 +39,5 @@
           <!-- <mesh filename="package://rotors_description/meshes/sonar_sensor/max_sonar_ez4.dae"/> -->
           <!--<mesh filename="package://ardupilot_sitl_gazebo_plugin/meshes/${sensor_mesh}"/>-->
-           <mesh filename="model://${sensor_mesh_scan}"/>
+           <mesh filename="file://${sensor_mesh_scan}"/>
          <!-- <mesh filename="package://ardupilot_sitl_gazebo_plugin/meshes/meshes_sensor/lidar_lite_v2/meshes/lidar_lite_v2.dae"/> -->
         </geometry>
@@ -54,5 +54,5 @@
         <always_on>true</always_on>
         <update_rate>${update_rate}</update_rate>
-        <pose>0 0 0 0 0 0</pose>
+        <pose>0 0 -0.004645 1.5707 0 0</pose>
         <visualize>true</visualize>
         <ray>
@@ -77,12 +77,9 @@
           </range>
         </ray>
-        <plugin name="gazebo_ros_${name}_controller" filename="librotors_gazebo_sonar_plugin.so">
-          <gaussianNoise>0.005</gaussianNoise>
-          <topicName>${ros_topic}</topicName>
-          <frameId>scan_link</frameId>
-        </plugin>
 	<plugin name="gazebo_ros_${name}_controller" filename="libgazebo_ros_laser.so">
+	<!--  <plugin name="gazebo_ros_${name}_controller" filename="libgazebo_ros_gpu_laser.so"> -->
           <topicName>/scan</topicName>
-          <frameName>scan_link</frameName>
+          <!-- <frameName>scan_link</frameName> -->
+	  <frameName>lidar_link</frameName>
 	</plugin>
       </sensor>

Commit message: [ARM-45]+[ARM-46]

File: Dev_code_version_SITL/ros_catkin_ws/src/ardupilot_sitl_gazebo_plugin/ardupilot_sitl_gazebo_plugin/urdf/armada.xacro (robot description, xacro)
@@ -7,5 +7,5 @@
   <xacro:property name="mesh_scale" value="1 1 1"/> <!-- 1 1 1 -->
   <xacro:property name="mesh_scale_prop" value="1 1 1"/>
-  <xacro:property name="mass" value="1.1" /> <!-- [kg] -->
+  <xacro:property name="mass" value="1.1" /> <!-- 1.1[kg] -->
   <xacro:property name="body_length" value="0.18" /> <!-- [m] 0.10 -->
   <xacro:property name="body_width" value="0.12" /> <!-- [m] 0.10 -->
@@ -31,5 +31,5 @@
   <!-- Property Blocks -->
   <xacro:property name="body_inertia">
-    <inertia ixx="0.0347563" ixy="0.0" ixz="0.0" iyy="0.0458929" iyz="0.0" izz="0.0977" /> <!-- [kg.m^2] [kg.m^2] [kg.m^2] [kg.m^2] [kg.m^2] [kg.m^2] -->
+    <inertia ixx="0.0347563" ixy="0.0" ixz="0.0" iyy="0.0458929" iyz="0.0" izz="0.0977" /> <!-- "0.0347563" ixy="0.0" ixz="0.0" iyy="0.0458929" iyz="0.0" izz="0.0977" [kg.m^2] [kg.m^2] [kg.m^2] [kg.m^2] [kg.m^2] [kg.m^2] -->
   </xacro:property>
   <!-- inertia of a single rotor, assuming it is a cuboid. Height=3mm, width=15mm -->
@@ -63,5 +63,5 @@
     name="lidar"
     parent="base_link"
-    update_rate="10"
+    update_rate="300"
     min_range="0.06"
     max_range="20.0"

File: Dev_code_version_SITL/ros_catkin_ws/src/ardupilot_sitl_gazebo_plugin/ardupilot_sitl_gazebo_plugin/urdf/armada_base.xacro (robot description, xacro)
@@ -78,5 +78,5 @@
     </plugin>
   </gazebo>
-   <xacro:if value="$(arg enable_ground_truth)">
+  <xacro:if value="$(arg enable_ground_truth)">
     <!-- Mount an IMU providing ground truth. -->
     <xacro:imu_plugin_macro
@@ -125,5 +125,5 @@
       image_scale=""
     >
-      <inertia ixx="0.00001" ixy="0.0" ixz="0.0" iyy="0.00001" iyz="0.0" izz="0.00001" /> --> <!-- [kg.m^2] [kg.m^2] [kg.m^2] [kg.m^2] [kg.m^2] [kg.m^2] -->
+      <inertia ixx="0.00001" ixy="0.0" ixz="0.0" iyy="0.00001" iyz="0.0" izz="0.00001" />  <!-- [kg.m^2] [kg.m^2] [kg.m^2] [kg.m^2] [kg.m^2] [kg.m^2] -->
       <origin xyz="0.0 0.0 0.0" rpy="0.0 0.0 0.0" />
     </xacro:odometry_plugin_macro>

File: Dev_code_version_SITL/ros_catkin_ws/src/ardupilot_sitl_gazebo_plugin/ardupilot_sitl_gazebo_plugin/urdf/sensors/lidar_sensor.urdf.xacro (robot description, xacro)
@@ -54,5 +54,5 @@
         <always_on>true</always_on>
         <update_rate>${update_rate}</update_rate>
-        <pose>0 0 -0.004645 1.5707 0 0</pose>
+        <pose>0 0 0 0 0 0</pose>
         <visualize>true</visualize>
         <ray>
